File: Light_Strip_Driver.kicad_pcb (KiCad board)
At the start: 2 copper layers, 36 parts, among them J1 LED_S2, J10 BUCK3_IN, J11 BUCK3_OUT, J2 LED_S1, J3 DC_PWR, J4 FAN_PWR, J5 FAN_PWR, J6 BUCK1_IN, J7 BUCK1_OUT, J8 BUCK2_IN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

Commit message: worked on pcb layout
Parts:
- U1: value LS20-X -> LSXX-X
- moved C3 120.1 mm to (83.9, 83.3)
- moved J3 120.1 mm to (80.0, 83.3)
- moved Q2 117.2 mm to (82.6, 98.1), turned to 90 degrees
- moved D1 117.0 mm to (85.7, 111.9)
- moved R3 117.0 mm to (74.7, 114.7)
- moved R1 117.0 mm to (78.8, 111.5)
- moved R2 117.0 mm to (78.8, 107.2)
- moved SW1 117.0 mm to (69.4, 109.4)
- moved R4 112.9 mm to (80.6, 102.5)
- moved J10 68.6 mm to (98.9, 99.2)
- moved D2 67.3 mm to (129.4, 79.8), turned to -90 degrees
- moved C2 65.8 mm to (105.6, 36.3)
- moved J1 65.6 mm to (103.9, 69.0)
- moved J2 65.6 mm to (108.5, 69.0)
- moved C1 65.5 mm to (105.6, 33.9)
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Routing:
- net Net-(SW10-A): track 0.00 -> 28.3 mm
- net Net-(SW4-A): track 0.00 -> 28.3 mm
- net Net-(SW7-A): track 0.00 -> 27.8 mm
- net VCC: track 0.00 -> 26.0 mm
- net Net-(A1-D3): track 0.00 -> 25.9 mm
- net +5V: track 0.00 -> 24.0 mm
- net +12V: track 37.9 -> 56.6 mm
- net Net-(SW1B-B): track 0.00 -> 17.4 mm
- net Net-(SW3-A): track 0.00 -> 17.2 mm
- net Net-(SW6-A): track 0.00 -> 16.9 mm
- net Net-(SW9-A): track 0.00 -> 16.6 mm
- net Net-(A1-D2): track 0.00 -> 14.9 mm
- net Net-(J7-Pin_1): track 0.00 -> 7.18 mm
- net Net-(J11-Pin_1): track 0.00 -> 7.17 mm
- net Net-(SW2-A): track 0.00 -> 6.65 mm
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
Commit message: finished pcb design
Parts:
- added D5: SB5x0, Diode_THT:D_DO-201AD_P12.70mm_Horizontal, F.Cu at (165.7, 70.9)
- added D6: SB5x0, Diode_THT:D_DO-201AD_P12.70mm_Horizontal, F.Cu at (171.6, 70.9)
- added D7: SB5x0, Diode_THT:D_DO-201AD_P12.70mm_Horizontal, F.Cu at (177.6, 70.9)
- added J12: BUCK4_IN, Connector_PinSocket_2.54mm:PinSocket_1x02_P2.54mm_Vertical, F.Cu at (131.9, 89.1)
- added J13: BUCK4_OUT, Connector_PinSocket_2.54mm:PinSocket_1x02_P2.54mm_Vertical, F.Cu at (164.5, 89.1)
- added J14: BUCK5_IN, Connector_PinSocket_2.54mm:PinSocket_1x02_P2.54mm_Vertical, F.Cu at (128.3, 89.1)
- added J15: BUCK5_OUT, Connector_PinSocket_2.54mm:PinSocket_1x02_P2.54mm_Vertical, F.Cu at (168.1, 89.1)
- added J16: BUCK6_IN, Connector_PinSocket_2.54mm:PinSocket_1x02_P2.54mm_Vertical, F.Cu at (124.7, 89.1)
- added J17: BUCK6_OUT, Connector_PinSocket_2.54mm:PinSocket_1x02_P2.54mm_Vertical, F.Cu at (171.7, 89.1)
- added REF**: LM2596_Buck_Module, Custom:LM2596_Buck_Module, F.Cu at (148.6, 105.9)
- added REF**: 23.5mmx17mm heatsink, Custom:23.5mmx17mm heatsink, F.Cu at (103.2, 103.8)
- added REF**: LM2596_Buck_Module, Custom:LM2596_Buck_Module, F.Cu at (148.6, 128.2)
- U1: value LSXX-X -> LS20-X
- moved J10 37.9 mm to (135.5, 89.1)
- moved J6 37.9 mm to (142.7, 89.1)
- moved J8 37.9 mm to (139.1, 89.1)
- moved D1 32.6 mm to (116.7, 121.8)
- moved R1 32.6 mm to (109.8, 121.4)
- moved R2 32.6 mm to (109.8, 117.1)
- moved R3 32.6 mm to (105.8, 124.5)
- moved SW1 32.6 mm to (100.5, 119.2)
- moved C1 31.2 mm to (136.6, 37.0)
- moved C2 31.2 mm to (136.6, 39.4)
- moved J2 31.1 mm to (139.6, 70.9)
- moved C3 31.1 mm to (114.9, 85.2)
- moved J3 31.1 mm to (111.0, 85.2)
- moved RV1 31.1 mm to (103.8, 67.7)
- moved SW2 31.1 mm to (146.4, 43.1)
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Routing:
- net +5V: track 24.0 -> 79.3 mm
- net VCC: track 26.0 -> 70.9 mm
- net +12V: track 56.6 -> 70.8 mm
- net Net-(J17-Pin_1): track 0.00 -> 8.22 mm
- net Net-(J15-Pin_1): track 0.00 -> 7.03 mm
- net Net-(SW1B-B): track 17.4 -> 11.0 mm
- net Net-(J13-Pin_1): track 0.00 -> 6.04 mm
- net Net-(J11-Pin_1): track 7.17 -> 6.09 mm
- net Net-(J7-Pin_1): track 7.18 -> 8.24 mm
- net Net-(J9-Pin_1): track 6.19 -> 7.07 mm
- net Net-(SW2-A): track 6.65 -> 5.79 mm
- net Net-(SW4-A): track 28.3 -> 27.5 mm
- net GND: vias 0 -> 4
- added copper zone on B.Cu, net GND
- added copper zone on F.Cu, net GND
Other:
- board outline added: 98.9 x 108.6 mm
- board text added: "<------- 75x75 Vesa Mounting ------->"
- board text added: "Buck Converter IN"
- board text added: "Buck Converter Out"
- board text added: "LS18"
- board text added: "LS19"
- board text added: "LS20"
